File: hardware/farm_hub/SILOAD REV A.kicad_pcb (KiCad board)
At the start: 2 copper layers, 59 x 36 mm, 11 parts, among them J1 XIAO_LEFT, J2 XIAO_RIGHT, J3 W5500_LEFT, J4 W5500_RIGHT

Commit message: Add dedicated 2-pin 5V/GND power connectors, update renders and production Gerbers
Parts:
- added J5: PWR_5V_IN, Connector_PinSocket_2.54mm:PinSocket_1x02_P2.54mm_Vertical, F.Cu at (63.5, 75.0)
Connections:
- J1 pad 2: unconnected-(J1-D1_GPIO2-Pad2) -> (no net)
- J1 pad 3: unconnected-(J1-D2_GPIO3-Pad3) -> (no net)
- J1 pad 4: unconnected-(J1-D3_GPIO4-Pad4) -> (no net)
- J1 pad 5: unconnected-(J1-D4_GPIO5-Pad5) -> (no net)
- J1 pad 6: unconnected-(J1-D5_GPIO6-Pad6) -> (no net)
- J2 pad 1: unconnected-(J2-5V_USB-Pad1) -> /+5V
- J4 pad 4: unconnected-(J4-NC-Pad4) -> (no net)
Routing:
- net /+5V: track 0.00 -> 84.0 mm
- net /+3V3: track 114.2 -> 66.5 mm
- net /SPI_MOSI: track 6.57 -> 20.2 mm
- net /SPI_MISO: track 35.5 -> 46.8 mm
- net /GND: track 124.2 -> 128.9 mm
- net /ETH_CSn: track 29.8 -> 30.9 mm
Other:
- board text added: "5V"
- board text added: "GND"
