File: hardware/farm_hub/SILOAD REV A.kicad_sch (KiCad schematic)
At the start: 6 parts, among them J1 XIAO_LEFT, J2 XIAO_RIGHT, J3 W5500_LEFT, J4 W5500_RIGHT

Commit message: Add dedicated 2-pin 5V/GND power connectors, update renders and production Gerbers
Parts:
- added J5: PWR_5V_IN, Connector_PinSocket_2.54mm:PinSocket_1x02_P2.54mm_Vertical, symbol SILOAD:J5_socket
Connections:
- net GND: now also J5.2 (GND)
- net +5V: now reaches J2.1 (5V_USB)
- net +5V: now also J5.1 (+5V_IN)
- no-connect marks 7 -> 6
