File: hardware/silo_unit/SILOAD LOAD CELL REV A.kicad_pcb (KiCad board)
At the start: 2 copper layers, 68 x 44 mm, 18 parts, among them J1 XIAO_LEFT, J2 XIAO_RIGHT, J3 HX711_MCU, J4 HX711_BRIDGE, J5 SENS1_LOADCELL, J6 SENS2_LOADCELL, J7 SENS3_LOADCELL, J8 SENS4_LOADCELL, J9 TEMP_DS18B20, U1 CD4052BE_MUX

Commit message: Place SiLoad logo vertically on left side of Silo Unit PCB for top-down visibility
Parts:
- LOGO1: value SiLoad badge 20mm -> SiLoad badge vertical; footprint SILOAD:SiLoad_Badge_20mm -> (none)
- moved LOGO1 41.4 mm to (53.4, 72.0)

Commit message: Add dedicated 2-pin 5V/GND power connectors, update renders and production Gerbers
Parts:
- added J10: PWR_5V_IN, Connector_PinSocket_2.54mm:PinSocket_1x02_P2.54mm_Vertical, F.Cu at (73.3, 75.5)
- moved C2 4.81 mm to (65.8, 76.5)
Connections:
- J1 pad 2: unconnected-(J1-D1_GPIO2-Pad2) -> (no net)
- J1 pad 3: unconnected-(J1-D2_GPIO3-Pad3) -> (no net)
- J1 pad 4: unconnected-(J1-D3_GPIO4-Pad4) -> (no net)
- J1 pad 5: unconnected-(J1-D4_GPIO5-Pad5) -> (no net)
- J1 pad 6: unconnected-(J1-D5_GPIO6-Pad6) -> (no net)
- J2 pad 1: unconnected-(J2-5V_USB-Pad1) -> /+5V
- J2 pad 5: unconnected-(J2-D9_GPIO8-Pad5) -> (no net)
- J4 pad 1: unconnected-(J4-B+-Pad1) -> (no net)
- J4 pad 2: unconnected-(J4-B--Pad2) -> (no net)
Routing:
- net /ONEWIRE_DQ: track 58.7 -> 27.8 mm, vias 0 -> 1
- net /+5V: track 0.00 -> 26.7 mm, vias 0 -> 2
- net /MUX_A: track 32.0 -> 26.2 mm, vias 1 -> 2
- net /+3V3: track 66.0 -> 68.0 mm, vias 2 -> 0
- net /GND: track 94.1 -> 92.4 mm, vias 4 -> 1
- net /LC_EP: track 57.5 -> 56.6 mm, vias 1 -> 3
- net /LC3_AP: track 29.7 -> 30.4 mm, vias 2 -> 1
- net /LC4_AN: track 23.9 -> 23.2 mm, vias 1 -> 0
Other:
- board text added: "5V"
