File: hardware/silo_unit/SILOAD LOAD CELL REV A.kicad_sch (KiCad schematic)
At the start: 13 parts, among them J1 XIAO_LEFT, J2 XIAO_RIGHT, J3 HX711_MCU, J4 HX711_BRIDGE, J5 SENS1_LOADCELL, J6 SENS2_LOADCELL, J7 SENS3_LOADCELL, J8 SENS4_LOADCELL, J9 TEMP_DS18B20, U1 CD4052BE_MUX

Commit message: Add dedicated 2-pin 5V/GND power connectors, update renders and production Gerbers
Parts:
- added J10: PWR_5V_IN, Connector_PinSocket_2.54mm:PinSocket_1x02_P2.54mm_Vertical, symbol SILOAD:J10_part
Connections:
- net GND: now also J10.2 (GND)
- net +5V: now reaches J2.1 (5V_USB)
- net +5V: now also J10.1 (+5V_IN)
- no-connect marks 9 -> 8
